File: eagle/avrReveil4/ardReveil4_tiny10.sch (EAGLE design)
At the start: 6 parts

Commit message: Minor edit
Parts:
- removed LED1: TLLY4400, led:TLLY4400
- added LED3: TLLY4400, led:TLLY4400
- R3: value 200+ -> 470
Connections:
- removed net 5V: R2.2
- new net N$6: R1.1, R2.2
- net GND: no longer R1.1
- net N$1: now also LED3.C; no longer LED1.C
- net N$3: now also LED3.A; no longer LED1.A
Other:
- note added: "PB1"
- moved on the sheet: R2
Changed lines of the file:
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@@
 <setting verticaltext="up"/>
 </settings>
-<grid distance="0.1" unitdist="inch" unit="inch" style="dots" multiple="1" display="yes" altdistance="0.01" altunitdist="inch" altunit="inch"/>
+<grid distance="0.1" unitdist="inch" unit="inch" style="lines" multiple="1" display="no" altdistance="0.01" altunitdist="inch" altunit="inch"/>
 <layers>
 <layer number="1" name="Top" color="4" fill="1" visible="no" active="no"/>
@@
 </classes>
 <parts>
-<part name="LED1" library="led" deviceset="TLLY4400" device="" value=""/>
 <part name="LED2" library="led" deviceset="TLLY4400" device="" value=""/>
 <part name="R1" library="resistor" deviceset="R-EU_" device="0204/7" value="1k"/>
 <part name="R2" library="resistor" deviceset="R-EU_" device="0204/7" value="1k"/>
-<part name="SUPPLY1" library="SparkFun-Aesthetics" deviceset="5V" device=""/>
-<part name="GND1" library="SparkFun-Aesthetics" deviceset="DGND" device=""/>
 <part name="LED_FLAME" library="led" deviceset="TLLY4400" device="" value=""/>
-<part name="R3" library="resistor" deviceset="R-EU_" device="0204/7" value="200+"/>
+<part name="R3" library="resistor" deviceset="R-EU_" device="0204/7" value="470"/>
 <part name="GND2" library="SparkFun-Aesthetics" deviceset="DGND" device=""/>
+<part name="LED3" library="led" deviceset="TLLY4400" device="" value=""/>
 </parts>
 <sheets>
@@
 <text x="53.34" y="76.2" size="1.27" layer="91">PB2</text>
 <text x="48.26" y="68.58" size="1.27" layer="91">PB0 (PWM)</text>
+<text x="53.34" y="73.66" size="1.27" layer="91">PB1</text>
 </plain>
 <instances>
-<instance part="LED1" gate="G$1" x="83.82" y="81.28"/>
 <instance part="LED2" gate="G$1" x="83.82" y="73.66"/>
 <instance part="R1" gate="G$1" x="83.82" y="63.5" rot="R90"/>
-<instance part="R2" gate="G$1" x="83.82" y="88.9" rot="R90"/>
-<instance part="SUPPLY1" gate="G$1" x="83.82" y="93.98"/>
-<instance part="GND1" gate="G$1" x="83.82" y="55.88"/>
+<instance part="R2" gate="G$1" x="93.98" y="63.5" rot="R270"/>
 <instance part="LED_FLAME" gate="G$1" x="66.04" y="66.04"/>
 <instance part="R3" gate="G$1" x="66.04" y="55.88" rot="R90"/>
 <instance part="GND2" gate="G$1" x="66.04" y="48.26"/>
+<instance part="LED3" gate="G$1" x="93.98" y="71.12" rot="R180"/>
 </instances>
 <busses>
@@
 <net name="N$1" class="0">
 <segment>
-<pinref part="LED1" gate="G$1" pin="C"/>
 <pinref part="LED2" gate="G$1" pin="A"/>
 <wire x1="83.82" y1="76.2" x2="58.42" y2="76.2" width="0.1524" layer="91"/>
+<pinref part="LED3" gate="G$1" pin="C"/>
+<wire x1="83.82" y1="76.2" x2="93.98" y2="76.2" width="0.1524" layer="91"/>
 </segment>
 </net>
@@
 </segment>
 </net>
-<net name="N$3" class="0">
-<segment>
-<pinref part="LED1" gate="G$1" pin="A"/>
-<pinref part="R2" gate="G$1" pin="1"/>
-</segment>
-</net>
-<net name="5V" class="0">
-<segment>
-<pinref part="R2" gate="G$1" pin="2"/>
-<pinref part="SUPPLY1" gate="G$1" pin="5V"/>
-</segment>
-</net>
 <net name="GND" class="0">
-<segment>
-<pinref part="R1" gate="G$1" pin="1"/>
-<pinref part="GND1" gate="G$1" pin="GND"/>
-</segment>
 <segment>
 <pinref part="R3" gate="G$1" pin="1"/>
@@
 </segment>
 </net>
+<net name="N$3" class="0">
+<segment>
+<pinref part="LED3" gate="G$1" pin="A"/>
+<pinref part="R2" gate="G$1" pin="1"/>
+</segment>
+</net>
+<net name="N$6" class="0">
+<segment>
+<pinref part="R2" gate="G$1" pin="2"/>
+<pinref part="R1" gate="G$1" pin="1"/>
+<wire x1="93.98" y1="58.42" x2="83.82" y2="58.42" width="0.1524" layer="91"/>
+<wire x1="58.42" y1="73.66" x2="78.74" y2="73.66" width="0.1524" layer="91"/>
+<wire x1="78.74" y1="73.66" x2="78.74" y2="58.42" width="0.1524" layer="91"/>
+<wire x1="78.74" y1="58.42" x2="83.82" y2="58.42" width="0.1524" layer="91"/>
+</segment>
+</net>
