File: eagle/DecadeCounterViewer/DecadeCounterViewer.brd (EAGLE design)
At the start: 34.8 x 28.4 mm, 5 parts, among them IC1 CD4017

Commit message: Added labels, reviewed. Ok for prod.
Parts:
- added R1: (no value), resistor:0204/7
Connections:
- net GND: now also R1.1
- net N$2: now also R1.2
Routing:
- net N$2: track 27.4 -> 32.7 mm
- net RES: track 53.0 -> 56.0 mm
- net N$14: track 7.45 -> 9.66 mm
- net N$17: track 18.7 -> 20.2 mm
- net N$18: track 17.0 -> 17.9 mm
- net VCC: track 45.5 -> 46.4 mm
- net N$16: track 18.0 -> 18.9 mm
- net N$13: track 13.3 -> 13.8 mm
Other:
- board text added: "Carry"
- board text added: "Clk"
- board text added: "GND"
- board text added: "Rst"
- board text added: "Vcc"
- board text added: "http://electrogeek.cc/decade counter viewer.html"
